Commit message: Added skied steering demo
Signed-off-by: Michał Pełka <michal.pelka@robotec.ai>

File: Assets/URDF/husky/husky.urdf (robot description, URDF)
Before this commit: robot husky_robot, 11 links, 10 joints
Links:
- link top_plate_link: geometry visual mesh filename=meshes/top_plate.dae
- link user_rail_link: geometry visual mesh filename=meshes/user_rail.dae
